Commit message: 210723 segway controller

File: src/robot_description/urdf/dual_motion_robot/dual_motion_robot.xacro (robot description, xacro)
@@ -8,12 +8,14 @@
     <!-- pose and inertial -->
     <inertial>
-      <mass value="0.001"/>
+      <mass value="118.1" />
       <origin rpy="0 0 0" xyz="0 0 0"/>
-      <inertia ixx="0.0395416666667" ixy="0" ixz="0" iyy="0.106208333333" iyz="0" izz="0.106208333333"/>
+      <inertia ixx="6.4387768" ixy="-0.0007626" ixz="-0.7441046"
+                iyy="46.1852065" iyz="-0.0011013"
+                izz="48.0676973" />
     </inertial>
     <!-- body -->
     <collision name="collision_chassis">
       <geometry>
-        <box size="0.7 0.7 0.07"/>
+        <box size="2.2 0.8 0.7"/>
       </geometry>
     </collision>
@@ -21,5 +23,5 @@
       <origin rpy="0 0 0" xyz="0 0 0"/>
       <geometry>
-        <box size="0.7 0.7 0.07"/>
+        <box size="2.2 0.8 0.7"/>
       </geometry>
       <material name="blue"/>
@@ -28,20 +30,21 @@
   <link name="wheel_link">
     <!-- pose and inertial -->
-    <pose>0 0 0.1 0 0 0</pose>
+    <pose>0 0 0 0 0 0</pose>
     <inertial>
-      <mass value="0.001"/>
-      <origin rpy="0 0 0" xyz="0 0 0.1"/>
-      <inertia ixx="0.0395416666667" ixy="0" ixz="0" iyy="0.106208333333" iyz="0" izz="0.106208333333"/>
+      <mass value="1"/>
+      <origin rpy="0 0 0" xyz="0 0 -0.35"/>
+      <inertia ixx="1" ixy="0" ixz="0" iyy="1" iyz="0" izz="1"/>
     </inertial>
     <!-- body -->
     <collision name="collision_wheel_link">
+      <origin rpy="0 0 0" xyz="0 0 -0.35"/>
       <geometry>
-        <box size="0.07 0.4 0.2"/>
+        <box size="0.1 1 0.1"/>
       </geometry>
     </collision>
     <visual>
-      <origin rpy="0 0 0" xyz="0 0 0"/>
+      <origin rpy="0 0 0" xyz="0 0 -0.35"/>
       <geometry>
-        <box size="0.07 0.4 0.2"/>
+        <box size="0.1 1 0.1"/>
       </geometry>
       <material name="blue"/>
@@ -49,8 +52,10 @@
   </link>
   <xacro:link_wheel name="link_right_wheel" />
-  <xacro:joint_wheel name="wheel_R_joint" child="link_right_wheel" origin_xyz="0 0.20 -0.1" />
+  <xacro:joint_wheel name="wheel_R_joint" child="link_right_wheel" origin_xyz="0 0.51 -0.35" origin_rpy="-3.14 0 0" />
+  <xacro:SimpleTransmissionVelocity n="0" joint="wheel_R_joint" />
   <xacro:link_wheel name="link_left_wheel" />
-  <xacro:joint_wheel name="wheel_L_joint" child="link_left_wheel" origin_xyz="0 -0.20 -0.1" />
-  <xacro:base_joint name="chassis_pos_joint" child="link_chassis" origin_xyz="0 0 0.11" />
-  <xacro:SimpleTransmissionPosition n="1" joint="chassis_pos_joint" />
+  <xacro:joint_wheel name="wheel_L_joint" child="link_left_wheel" origin_xyz="0 -0.51 -0.35" origin_rpy="0 0 0" />
+  <xacro:SimpleTransmissionVelocity n="1" joint="wheel_L_joint" />
+  <xacro:base_joint name="chassis_pos_joint" child="link_chassis" origin_xyz="0 0 0.0" />
+  <xacro:SimpleTransmissionPosition n="2" joint="chassis_pos_joint" />
 </robot>

File: src/robot_description/urdf/dual_motion_robot/dual_motion_robot_transmision.xacro (robot description, xacro)
@@ -15,12 +15,12 @@
   </xacro:macro>
   <!-- Transmission macro -->
-  <xacro:macro name="SimpleTransmissionEffort" params="joint n">
+  <xacro:macro name="SimpleTransmissionVelocity" params="joint n">
     <transmission name="tran${n}">
       <type>transmission_interface/SimpleTransmission</type>
       <joint name="${joint}">
-        <hardwareInterface>hardware_interface/EffortJointInterface</hardwareInterface>
+        <hardwareInterface>hardware_interface/VelocityJointInterface</hardwareInterface>
       </joint>
       <actuator name="motor${n}">
-        <hardwareInterface>hardware_interface/EffortJointInterface</hardwareInterface>
+        <hardwareInterface>hardware_interface/VelocityJointInterface</hardwareInterface>
         <mechanicalReduction>1</mechanicalReduction>
       </actuator>

File: src/robot_description/urdf/dual_motion_robot/macros.xacro (robot description, xacro)
@@ -4,12 +4,14 @@
         <link name="${name}">
             <inertial>
-              <mass value="0.2"/>
+              <mass value="3.871" />
               <origin rpy="0 1.5707 1.5707" xyz="0 0 0"/>
-              <inertia ixx="0.000526666666667" ixy="0" ixz="0" iyy="0.000526666666667" iyz="0" izz="0.001"/>
+              <inertia ixx="0.056425" ixy="0.0" ixz="0.0"
+                      iyy="0.094098" iyz="0.0"
+                      izz="0.056425" />
             </inertial>
             <collision name="link_right_wheel_collision">
               <origin rpy="0 1.5707 1.5707" xyz="0 0 0"/>
               <geometry>
-                <cylinder length="0.04" radius="0.1"/>
+                <cylinder length="0.14" radius="0.2"/>
               </geometry>
             </collision>
@@ -17,16 +19,16 @@
               <origin rpy="0 1.5707 1.5707" xyz="0 0 0"/>
               <geometry>
-                <cylinder length="0.04" radius="0.1"/>
+                <cylinder length="0.14" radius="0.2"/>
               </geometry>
             </visual>
         </link>
     </xacro:macro>
-    <xacro:macro name="joint_wheel" params="name child origin_xyz">
+    <xacro:macro name="joint_wheel" params="name child origin_xyz origin_rpy">
       <joint name="${name}" type="continuous">
-        <origin rpy="0 0 0" xyz="${origin_xyz}"/>
+        <origin rpy="${origin_rpy}" xyz="${origin_xyz}"/>
         <child link="${child}"/>
         <parent link="wheel_link"/>
         <axis rpy="0 0 0" xyz="0 1 0"/>
-        <limit effort="10000" velocity="1000"/>
+        <!--limit effort="10000" velocity="100"/-->
         <joint_properties damping="1.0" friction="1.0"/>
       </joint>

File: src/robot_description/urdf/kitech_segway/kitech_segway_stl.xacro (robot description, xacro)
@@ -1,4 +1,5 @@
 <?xml version="1.0"?>
 <robot name="kitech_segway_type" xmlns:xacro="http://ros.org/wiki/xacro">
+  <xacro:include filename="$(find robot_description)/urdf/kitech_segway/materials.xacro" />
   <xacro:property name="deg_to_rad" value="0.01745329251994329577"/>
   <!-- Constants -->
@@ -52,5 +53,5 @@
     <collision>
       <geometry>
-	      <box size="2.2 0.7 0.8"/>
+	      <box size="2.2 0.7 0.2"/>
       </geometry>
       <origin rpy="${90.*M_PI/180.} 0 0" xyz="0 0 0.45"/>
@@ -58,5 +59,5 @@
     <inertial>
       <origin xyz="0 0 0" rpy="0 0 0"/>
-      <mass value="10"/>
+      <mass value="20"/>
       <inertia ixx="2.2124416e-03" ixy="-1.2294101e-05" ixz="3.4938785e-05"
                iyy="2.1193702e-03" iyz="-5.0120904e-06"
@@ -66,5 +67,5 @@
   <gazebo reference="base_link">
     <turnGravityOff>false</turnGravityOff>
-    <material>Gazebo/Gray</material>
+    <material>Gazebo/Darkgreen</material>
   </gazebo>
   <link name="mp_left_wheel">
@@ -83,5 +84,5 @@
     <inertial>
       <origin xyz="0 0 0" rpy="0 0 0"/>
-      <mass value="10"/>
+      <mass value="5"/>
       <inertia ixx="2.2124416e-03" ixy="-1.2294101e-05" ixz="3.4938785e-05"
                iyy="2.1193702e-03" iyz="-5.0120904e-06"
@@ -91,5 +92,5 @@
   <gazebo reference="mp_left_wheel">
     <turnGravityOff>false</turnGravityOff>
-    <material>Gazebo/Black</material>
+    <material>Gazebo/DarkGrey</material>
   </gazebo>
   <joint name="mp_left_wheel_joint" type="continuous">
@@ -114,5 +115,5 @@
     <inertial>
       <origin xyz="0 0 0" rpy="0 0 0"/>
-      <mass value="10"/>
+      <mass value="5"/>
       <inertia ixx="2.2124416e-03" ixy="-1.2294101e-05" ixz="3.4938785e-05"
                iyy="2.1193702e-03" iyz="-5.0120904e-06"
@@ -122,5 +123,5 @@
   <gazebo reference="mp_right_wheel">
     <turnGravityOff>false</turnGravityOff>
-    <material>Gazebo/Black</material>
+    <material>Gazebo/DarkGrey</material>
   </gazebo>
   <joint name="mp_right_wheel_joint" type="continuous">

File: src/robot_description/urdf/kitech_segway/materials.xacro (robot description, xacro)
@@ -26,5 +26,5 @@
   </material>
   <material name="darkgreen">
-    <color rgba="0 1.0 0 1.0"/>
+    <color rgba="0 0.3 0 1.0"/>
   </material>
 </robot>

Commit message: 210726 edit xacro

File: src/robot_description/urdf/dual_motion_robot/dual_motion_robot.xacro (robot description, xacro)
@@ -11,6 +11,6 @@
       <origin rpy="0 0 0" xyz="0 0 0"/>
       <inertia ixx="6.4387768" ixy="-0.0007626" ixz="-0.7441046"
-                iyy="46.1852065" iyz="-0.0011013"
-                izz="48.0676973" />
+          iyy="46.1852065" iyz="-0.0011013"
+          izz="48.0676973" />
     </inertial>
     <!-- body -->
@@ -30,9 +30,8 @@
   <link name="wheel_link">
     <!-- pose and inertial -->
-    <pose>0 0 0 0 0 0</pose>
     <inertial>
       <mass value="1"/>
       <origin rpy="0 0 0" xyz="0 0 -0.35"/>
-      <inertia ixx="1" ixy="0" ixz="0" iyy="1" iyz="0" izz="1"/>
+      <inertia ixx="0.01" ixy="0" ixz="0" iyy="0.01" iyz="0" izz="0.01"/>
     </inertial>
     <!-- body -->
@@ -52,9 +51,9 @@
   </link>
   <xacro:link_wheel name="link_right_wheel" />
-  <xacro:joint_wheel name="wheel_R_joint" child="link_right_wheel" origin_xyz="0 0.51 -0.35" origin_rpy="-3.14 0 0" />
-  <xacro:SimpleTransmissionVelocity n="0" joint="wheel_R_joint" />
+  <xacro:joint_wheel name="wheel_R_joint" child="link_right_wheel" origin_xyz="0 0.51 -0.35" origin_rpy="0 0 0" />
+  <xacro:SimpleTransmissionEffort n="0" joint="wheel_R_joint" />
   <xacro:link_wheel name="link_left_wheel" />
   <xacro:joint_wheel name="wheel_L_joint" child="link_left_wheel" origin_xyz="0 -0.51 -0.35" origin_rpy="0 0 0" />
-  <xacro:SimpleTransmissionVelocity n="1" joint="wheel_L_joint" />
+  <xacro:SimpleTransmissionEffort n="1" joint="wheel_L_joint" />
   <xacro:base_joint name="chassis_pos_joint" child="link_chassis" origin_xyz="0 0 0.0" />
   <xacro:SimpleTransmissionPosition n="2" joint="chassis_pos_joint" />

File: src/robot_description/urdf/dual_motion_robot/dual_motion_robot_transmision.xacro (robot description, xacro)
@@ -27,3 +27,15 @@
     </transmission>
   </xacro:macro>
+  <xacro:macro name="SimpleTransmissionEffort" params="joint n">
+    <transmission name="tran${n}">
+      <type>transmission_interface/SimpleTransmission</type>
+      <joint name="${joint}">
+        <hardwareInterface>hardware_interface/EffortJointInterface</hardwareInterface>
+      </joint>
+      <actuator name="motor${n}">
+        <hardwareInterface>hardware_interface/EffortJointInterface</hardwareInterface>
+        <mechanicalReduction>1</mechanicalReduction>
+      </actuator>
+    </transmission>
+  </xacro:macro>
 </robot>

File: src/robot_description/urdf/dual_motion_robot/macros.xacro (robot description, xacro)
@@ -30,5 +30,5 @@
         <parent link="wheel_link"/>
         <axis rpy="0 0 0" xyz="0 1 0"/>
-        <!--limit effort="10000" velocity="100"/-->
+        <limit effort="1" velocity="100"/>
         <joint_properties damping="1.0" friction="1.0"/>
       </joint>

Commit message: 210727 model debuging

File: src/robot_description/urdf/dual_motion_robot/dual_motion_robot.xacro (robot description, xacro)
@@ -50,11 +50,11 @@
     </visual>
   </link>
+  <xacro:link_wheel name="link_left_wheel" />
+  <xacro:joint_wheel name="wheel_L_joint" child="link_left_wheel" origin_xyz="0 0.51 -0.35" origin_rpy="0 0 0" />
+  <xacro:SimpleTransmissionVelocity n="0" joint="wheel_L_joint" />
   <xacro:link_wheel name="link_right_wheel" />
-  <xacro:joint_wheel name="wheel_R_joint" child="link_right_wheel" origin_xyz="0 0.51 -0.35" origin_rpy="0 0 0" />
-  <xacro:SimpleTransmissionEffort n="0" joint="wheel_R_joint" />
-  <xacro:link_wheel name="link_left_wheel" />
-  <xacro:joint_wheel name="wheel_L_joint" child="link_left_wheel" origin_xyz="0 -0.51 -0.35" origin_rpy="0 0 0" />
-  <xacro:SimpleTransmissionEffort n="1" joint="wheel_L_joint" />
+  <xacro:joint_wheel name="wheel_R_joint" child="link_right_wheel" origin_xyz="0 -0.51 -0.35" origin_rpy="0 0 0" />
+  <xacro:SimpleTransmissionVelocity n="1" joint="wheel_R_joint" />
   <xacro:base_joint name="chassis_pos_joint" child="link_chassis" origin_xyz="0 0 0.0" />
-  <xacro:SimpleTransmissionPosition n="2" joint="chassis_pos_joint" />
+  <xacro:SimpleTransmissionEffort n="2" joint="chassis_pos_joint" />
 </robot>

File: src/robot_description/urdf/dual_motion_robot/macros.xacro (robot description, xacro)
@@ -30,5 +30,5 @@
         <parent link="wheel_link"/>
         <axis rpy="0 0 0" xyz="0 1 0"/>
-        <limit effort="1" velocity="100"/>
+        <limit effort="1000" velocity="100"/>
         <joint_properties damping="1.0" friction="1.0"/>
       </joint>
@@ -45,5 +45,6 @@
         <parent link="wheel_link"/>
         <axis rpy="0 0 0" xyz="1 0 0"/>
-        <limit effort="10" lower="-0.35" upper="0.35" velocity="0.1" />
+        <limit effort="10000" lower="-0.35" upper="0.35" velocity="0.1" />
+        <joint_properties damping="1.0" friction="1.0"/>
       </joint>
     </xacro:macro>

Commit message: 210730 controller dubuging

File: src/robot_description/urdf/dual_motion_robot/dual_motion_robot.xacro (robot description, xacro)
@@ -8,5 +8,6 @@
     <!-- pose and inertial -->
     <inertial>
-      <mass value="118.1" />
+      <mass value="1" />
+      <!--mass value="118.1" /-->
       <origin rpy="0 0 0" xyz="0 0 0"/>
       <inertia ixx="6.4387768" ixy="-0.0007626" ixz="-0.7441046"
@@ -23,5 +24,6 @@
       <origin rpy="0 0 0" xyz="0 0 0"/>
       <geometry>
-        <box size="2.2 0.8 0.7"/>
+        <mesh filename="package://robot_description/mesh/for_VREP/Body_with_wheel_plate.stl" scale="0.001 0.001 0.001"/>
+        <!--box size="2.2 0.8 0.7"/-->
       </geometry>
       <material name="blue"/>

File: src/robot_description/urdf/dual_motion_robot/macros.xacro (robot description, xacro)
@@ -17,7 +17,8 @@
             </collision>
             <visual name="${name}_visual">
-              <origin rpy="0 1.5707 1.5707" xyz="0 0 0"/>
+              <origin rpy="0 0 0" xyz="0 0 0"/>
               <geometry>
-                <cylinder length="0.14" radius="0.2"/>
+                <mesh filename="package://robot_description/mesh/for_VREP/Wheel.stl" scale="0.001 0.001 0.001"/>
+                <!--cylinder length="0.14" radius="0.2"/-->
               </geometry>
             </visual>
@@ -45,5 +46,5 @@
         <parent link="wheel_link"/>
         <axis rpy="0 0 0" xyz="1 0 0"/>
-        <limit effort="10000" lower="-0.35" upper="0.35" velocity="0.1" />
+        <limit effort="10000" lower="-1" upper="1" velocity="0.01" />
         <joint_properties damping="1.0" friction="1.0"/>
       </joint>
